File: DrinkbotPCB.sch (EAGLE design)
At the start: 35 parts, among them IC1 L7805, J1 POWER_JACKPTH, Q1 MOSFET-NCHANNELFQP30N06L, Q2 MOSFET-NCHANNELFQP30N06L, Q3 MOSFET-NCHANNELFQP30N06L, Q4 MOSFET-NCHANNELFQP30N06L, Q5 MOSFET-NCHANNELFQP30N06L, Q6 MOSFET-NCHANNELFQP30N06L, Q7 MOSFET-NCHANNELFQP30N06L, Q8 MOSFET-NCHANNELFQP30N06L

Commit message: Updated Schematics/Gerbers/Board Layout
Parts:
- added C1, C2: 10uF, SparkFun-Passives:CAP_POLPTH2
- added C3, C4: 22pf, SparkFun-Capacitors:CAPKIT
- added C5, C6: 0.1uF, SparkFun-Capacitors:CAPKIT
- added D9: 1N4007, SparkFun-DiscreteSemi:DIODEPTH
- added EXTRA-5V: (no value), SparkFun-Connectors:M05PTH
- added JP1: RGBLED1, SparkFun-Connectors:M03JST-PTH
- added JP3: ISP, SparkFun-Connectors:M03X2
- added JP4: ALCOHOL, SparkFun-Connectors:M04PTH
- added Q10, Q9: BSS138, SparkFun-DiscreteSemi:MOSFET-NCHANNELBSS138
- added R10, R11, R12, R13, R14, R15, R9: 10k, SparkFun-Resistors:RESISTORPTH-1/6W
- added U$1: SPARK-CORE, Spark:SPARK_CORE
- added U$2: TMP, SparkFun-Sensors:TEMPERATURE-SENSOR
- added U1: ATMEGA328P, SparkFun-DigitalIC:ATMEGA328_SMT
- added U2: TXB0108, adafruit:TXB0108PWR
- added Y1: 16Mhz, SparkFun-FreqCtrl:CRYSTALHC49US
- GPIO_HEADER1: value RPI_GPIO_HEADER -> RPI-GPIO
- IC1: value L7805 -> L7805-5V
- J1: value POWER_JACKPTH -> 12V-PWR
- Q1, Q2, Q3, Q4, Q5, Q6, Q7, Q8: value MOSFET-NCHANNELFQP30N06L -> FQP30N06L
- R1, R2, R3, R4, R5, R6, R7, R8: device SparkFun-Passives:RESISTORPTH-1/4W -> SparkFun-Resistors:RESISTORPTH-1/6W
Connections:
- new net +3V3: C6.1, Q10.G, Q9.G, R11.1, R14.1, R9.1, U$1.VCC, U$2.VCC, U2.VCCA
- new net AP0: U1.PC0(ADC0), UNIT0.6
- new net AP1: U1.PC1(ADC1), UNIT1.6
- new net AP2: U1.PC2(ADC2), UNIT2.6
- new net AP3: U1.PC3(ADC3), UNI3.6
- new net AP4: U1.PC4(ADC4/SDA), UNIT4.6
- new net AP5: U1.PC5(ADC5/SCL), UNIT5.6
- new net AP6: U1.ADC6, UNIT6.6
- new net AP7: U1.ADC7, UNIT7.6
- new net AS2-3V: U$1.A2, U2.A4
- new net AS2-5V: JP4.2, U2.B4
- new net AS3V: U$1.A3, U2.A3
- new net AS5V: R15.1, U2.B3
- new net AT-RX: U1.PD0(RXD), U2.B1
- new net AT-TX: U1.PD1(TXD), U2.B2
- new net DP0: U1.PB0(ICP), UNIT0.7
- new net DP1: U1.PB1(OC1A), UNIT1.7
- new net DP2: U1.PD2(INT0), UNIT2.7
- new net DP3: U1.PD3(INT1), UNI3.7
- new net DP4: U1.PD4(XCK/T0), UNIT4.7
- new net DP5: U1.PD5(T1), UNIT5.7
- new net DP6: U1.PD6(AIN0), UNIT6.7
- new net DP7: U1.PD7(AIN1), UNIT7.7
- new net EXTRA1-3V3: U$1.D2, U2.A5
- new net EXTRA1-5V: EXTRA-5V.4, U2.B5
- new net EXTRA2-3V3: U$1.D5, U2.A6
- new net EXTRA2-5V: EXTRA-5V.3, U2.B6
- new net EXTRA3-3V3: U$1.D6, U2.A7
- new net EXTRA3-5V: EXTRA-5V.2, U2.B7
- new net HV1: JP1.3, Q9.D, R10.2
- new net LEDIN0: Q10.D, R13.2, UNIT0.3
- new net LEDOUT0: UNIT0.4, UNIT1.3
- new net LEDOUT1: UNIT1.4, UNIT2.3
- new net LEDOUT2: UNI3.3, UNIT2.4
- new net LEDOUT3: UNI3.4, UNIT4.3
- new net LEDOUT4: UNIT4.4, UNIT5.3
- new net LEDOUT5: UNIT5.4, UNIT6.3
- new net LEDOUT6: UNIT6.4, UNIT7.3
- new net LEDOUT7: UNIT7.4
- new net LV-RX: GPIO_HEADER1G$1.GPIO$16, U$1.RX, U2.A2
- new net LV-TX: GPIO_HEADER1G$1.GPIO$15, U$1.TX, U2.A1
- new net MISO: JP3.1, U1.PB4(MISO)
- new net MOSI: JP3.4, U1.PB3(MOSI/OC2)
- new net N$1: C1.+, D9.C, IC1.IN
- new net N$2: C3.2, U1.PB6(XTAL1/TOSC1), Y1.2
- new net N$3: C4.2, U1.PB7(XTAL2/TOSC2), Y1.1
- new net N$5: R14.2, U2.OE
- new net N$7: JP4.3, R15.2
- new net PUMPLEDS: GPIO_HEADER1G$1.GPIO$10, Q10.S, R9.2, U$1.D3
- new net RESET: JP3.5, R12.2, U1.PC6(/RESET)
- new net RGBLED1: Q9.S, R11.2, U$1.D7
- new net SCK: JP3.3, U1.PB5(SCK)
- new net TEMPSENSOR1: U$1.D4, U$2.ADJ
- net +5V: now also C2.+, C5.1, EXTRA-5V.5, JP1.1, JP3.2, JP4.1, R10.1, R12.1, R13.1, U$1.RAW, U1.AREF, U1.AVCC, U1.VCC@1, U1.VCC@2, U2.VCCB, UNI3.2, UNIT0.2, UNIT1.2, UNIT2.2, UNIT4.2, UNIT5.2, UNIT6.2, UNIT7.2
- net GND: now also C1.-, C2.-, C3.1, C4.1, C5.2, C6.2, EXTRA-5V.1, JP1.2, JP3.6, JP4.4, U$1.GND@2, U$1.GND@21, U$2.GND, U1.AGND, U1.GND@1, U1.GND@2, U2.GND, UNI3.5, UNIT0.5, UNIT1.5, UNIT2.5, UNIT4.5, UNIT5.5, UNIT6.5, UNIT7.5
- net PUMP0: now also R3.1, U$1.D0; no longer R1.1
- net PUMP1: now also U$1.D1
- net PUMP2: now also R1.1, U$1.A0; no longer R3.1
- net PUMP3: now also U$1.A1
- net PUMP4: now also U$1.A4
- net PUMP5: now also U$1.A5
- net PUMP6: now also U$1.A6
- net PUMP7: now also U$1.A7
- net VIN12: now also D9.A; no longer IC1.IN
